File: 13A-Pro.kicad_pcb (KiCad board)
At the start: 2 copper layers, 81 x 81 mm, 30 parts, among them SW1 SW_Push, U1 ProMicro

Commit message: PCB Update ver 1.0
Parts:
- moved SW1 5.18 mm to (146.8, 75.4), turned to 90 degrees
- moved U1 4.39 mm to (146.8, 76.2)
Connections:
- U1 pad 10: COL1 -> COL2
- U1 pad 11: COL2 -> COL1
- U1 pad 5: ROW3 -> ROW0
- U1 pad 6: ROW2 -> ROW1
- U1 pad 7: ROW1 -> ROW2
- U1 pad 8: ROW0 -> ROW3
Routing:
- net COL1: track 0.00 -> 137.1 mm
- net COL0: track 0.00 -> 133.2 mm
- net COL2: track 0.00 -> 86.2 mm
- net ROW3: track 57.1 -> 128.4 mm
- net ROW2: track 57.2 -> 105.3 mm
- net COL3: track 0.00 -> 35.5 mm
- net GND: track 0.00 -> 31.2 mm
- net ROW1: track 38.1 -> 64.8 mm
- net ROW0: track 38.1 -> 49.1 mm
- net Net-(U1-RST): track 0.00 -> 9.67 mm
- added copper zone on B.Cu, net GND
- added copper zone on F.Cu, net GND
Other:
- board text added: "HARD RESET >>>"
- board text added: "MADE BY RELREL___"
- board text added: "TO INFINITY AND BEYOND."
